File: pcb_car/tracking_v2.sch (KiCad schematic (older format))
At the start: 20 parts, among them J1 Conn_01x02, J2 Conn_01x20_Female, J3 Conn_01x20_Female, J4 Conn_01x02, J5 Conn_01x02, J6 Conn_01x02, J7 Conn_01x02, J8 Conn_01x03, J9 Conn_01x03, SW1 SW_Push, U1 GY-521, U2 L293D, U3 L293D

Commit message: pcb car
updated schematic and libraries
Parts:
- added R10, R11, R4, R5, R6, R7, R8, R9: R, Resistors_SMD:R_1206_HandSoldering, symbol R
Connections:
- net 5V: now also U3.16 (VS); no longer U3.8 (VS)
- net BATT: now also U3.8 (VS); no longer U3.16 (VS)
- net GND: now also R2.1, R10.1, R11.2, R4.2, R5.1, R6.2, R7.1, R8.2, R9.2; no longer R2.2
- net EN1_A: now reaches J2.9 (Pin_9), U2.1 (enable_1)
- net IN3_A: now reaches J2.13 (Pin_13), U2.10 (INPUT_3)
- net IN3_A: now also R8.1
- net IN4_A: now reaches J2.12 (Pin_12), U2.15 (INPUT_4)
- net IN4_A: now also R7.2
- net IN1_A: now reaches J2.10 (Pin_10), U2.2 (input_1)
- net IN1_A: now also R2.2
- net IN2_A: now reaches J2.11 (Pin_11), U2.7 (INPUT_2)
- net IN2_A: now also R4.1
- net EN2_A: now reaches J2.14 (Pin_14), U2.9 (ENABLE_1)
- net at J2.5 (Pin_5), SW1.1: now also R9.1; no longer R2.1
- net DATA1: now reaches J3.4 (Pin_4), J9.2 (Pin_2)
- net DATA2: now reaches J3.2 (Pin_2), J8.2 (Pin_2)
- net IN3_B: now reaches J3.10 (Pin_10), U3.10 (INPUT_3)
- net IN3_B: now also R11.1
- net EN2_B: now reaches J3.11 (Pin_11), U3.9 (ENABLE_1)
- net IN2_B: now reaches J3.12 (Pin_12), U3.7 (INPUT_2)
- net IN2_B: now also R6.1
- net IN1_B: now reaches J3.5 (Pin_5), U3.2 (input_1)
- net IN1_B: now also R5.2
- net EN1_B: now reaches J3.6 (Pin_6), U3.1 (enable_1)
- net IN4_B: now reaches J3.7 (Pin_7), U3.15 (INPUT_4)
- net IN4_B: now also R10.2
- no-connect marks 16 -> 20
Other:
- moved on the sheet: C1, D1, D2, J1, J2, J3, J4, J5, J6, J7, J8, J9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

Commit message: Added second iteration of PCB design (incomplete), moved libraries to subfolder
Parts:
- removed J2: Conn_01x20_Female, Socket_Strips:Socket_Strip_Straight_1x20_Pitch2.54mm, symbol Conn_01x20_Female
- added J5: Conn_01x16_Female, Socket_Strips:Socket_Strip_Straight_1x16_Pitch2.54mm, symbol Conn_01x16_Female
- renumbered J4 to J2, J6 to J3, J7 to J4, J5 to J6, J3 to J7, R4 to R3, R5 to R4, R6 to R5, R7 to R6, R8 to R7, R9 to R8, R3 to R9, U2 to U1, U3 to U2, U1 to U3
Connections:
- net labels added: 3v3_gyro
- no-connect marks 20 -> 16
Changed lines of the file:
@@
 LIBS:contrib
 LIBS:valves
-LIBS:gy-521
 LIBS:L293D
 LIBS:wemos
+LIBS:gy-521
 LIBS:tracking_v2-cache
 EELAYER 25 0
@@
 NoConn ~ 6185 4065
 $Comp
-L GY-521 U1
+L GY-521 U3
 U 1 1 5B033AEE
 P 4805 3225
-F 0 "U1" H 4905 3575 60  0000 C CNN
+F 0 "U3" H 4905 3575 60  0000 C CNN
 F 1 "GY-521" H 5005 3675 60  0000 C CNN
 F 2 "GY-521:GY-521" H 4805 3225 60  0001 C CNN
@@
 $EndComp
 $Comp
-L Conn_01x02 J5
+L Conn_01x02 J6
 U 1 1 5B034C51
 P 5805 1840
-F 0 "J5" H 5805 1940 50  0000 C CNN
+F 0 "J6" H 5805 1940 50  0000 C CNN
 F 1 "Conn_01x02" H 5805 1640 50  0000 C CNN
 F 2 "Pin_Headers:Pin_Header_Straight_1x02_Pitch2.54mm" H 5805 1840 50  0001 C CNN
@@
 $EndComp
 $Comp
-L Conn_01x02 J6
+L Conn_01x02 J3
 U 1 1 5B034DEC
 P 3635 1585
-F 0 "J6" H 3635 1685 50  0000 C CNN
+F 0 "J3" H 3635 1685 50  0000 C CNN
 F 1 "Conn_01x02" H 3635 1385 50  0000 C CNN
 F 2 "Pin_Headers:Pin_Header_Straight_1x02_Pitch2.54mm" H 3635 1585 50  0001 C CNN
@@
 $EndComp
 $Comp
-L L293D U2
+L L293D U1
 U 1 1 5B03538E
 P -6415 13260
-F 0 "U2" H -6315 13510 60  0000 C CNN
-F 1 "L293D" H -6315 13510 60  0000 C CNN
+F 0 "U1" H -6365 13310 60  0000 C CNN
+F 1 "L293D" H 2915 19610 60  0000 C CNN
 F 2 "L293D:DIL16" H -6415 13260 60  0001 C CNN
 F 3 "" H -6415 13260 60  0001 C CNN
@@
 BATT
 $Comp
-L Conn_01x02 J7
+L Conn_01x02 J4
 U 1 1 5B036CAE
 P 3885 6095
-F 0 "J7" H 3885 6195 50  0000 C CNN
+F 0 "J4" H 3885 6195 50  0000 C CNN
 F 1 "Conn_01x02" H 3885 5895 50  0000 C CNN
 F 2 "Pin_Headers:Pin_Header_Straight_1x02_Pitch2.54mm" H 3885 6095 50  0001 C CNN
@@
 $EndComp
 $Comp
-L Conn_01x02 J4
+L Conn_01x02 J2
 U 1 1 5B03776A
 P 1420 5965
-F 0 "J4" H 1420 6065 50  0000 C CNN
+F 0 "J2" H 1420 6065 50  0000 C CNN
 F 1 "Conn_01x02" H 1420 5765 50  0000 C CNN
 F 2 "Pin_Headers:Pin_Header_Straight_1x02_Pitch2.54mm" H 1420 5965 50  0001 C CNN
@@
 $EndComp
 $Comp
-L R R3
+L R R9
 U 1 1 5B038425
 P 5585 5720
-F 0 "R3" V 5665 5720 50  0000 C CNN
+F 0 "R9" V 5665 5720 50  0000 C CNN
 F 1 "R" V 5585 5720 50  0000 C CNN
 F 2 "Resistors_SMD:R_1206_HandSoldering" V 5515 5720 50  0001 C CNN
@@
 3V3
 Wire Wire Line
-	4205 3225 4205 5065
-Wire Wire Line
-	4205 5065 5085 5065
-Wire Wire Line
 	5405 3225 5405 3775
 Wire Wire Line
@@
 	3560 6010 3560 6160
 Wire Wire Line
-	3610 6160 3485 6160
+	3485 6160 3610 6160
 Connection ~ 3560 6160
 Wire Wire Line
@@
 	1915 6010 1915 6160
 Wire Wire Line
-	1985 6160 1885 6160
+	1885 6160 1985 6160
 Connection ~ 1915 6160
 Wire Wire Line
@@
 	1220 6310 1985 6310
 Wire Wire Line
-	1270 1115 1270 1030
+	1270 1030 1270 1115
 Wire Wire Line
 	1370 1115 1370 1055
@@
 Connection ~ 1270 1060
 $Comp
-L Conn_01x20_Female J3
+L Conn_01x20_Female J7
 U 1 1 5B03D2A3
 P 6085 4265
-F 0 "J3" H 6085 5265 50  0000 C CNN
+F 0 "J7" H 6085 5265 50  0000 C CNN
 F 1 "Conn_01x20_Female" H 6085 3165 50  0000 C CNN
 F 2 "Socket_Strips:Socket_Strip_Straight_1x20_Pitch2.54mm" H 6085 4265 50  0001 C CNN
@@
 $EndComp
 $Comp
-L Conn_01x20_Female J2
-U 1 1 5B03D59A
-P 5985 4865
-F 0 "J2" H 5985 5865 50  0000 C CNN
-F 1 "Conn_01x20_Female" H 5985 3765 50  0000 C CNN
-F 2 "Socket_Strips:Socket_Strip_Straight_1x20_Pitch2.54mm" H 5985 4865 50  0001 C CNN
-F 3 "" H 5985 4865 50  0001 C CNN
-	1    5985 4865
-	0    -1   -1   0
-$EndComp
-$Comp
-L L293D U3
+L L293D U2
 U 1 1 5B03F194
 P -4295 8820
-F 0 "U3" H -4195 9070 60  0000 C CNN
-F 1 "L293D" H -4195 9070 60  0000 C CNN
+F 0 "U2" H -4245 8870 60  0000 C CNN
+F 1 "L293D" H 4565 16775 60  0000 C CNN
 F 2 "L293D:DIL16" H -4295 8820 60  0001 C CNN
 F 3 "" H -4295 8820 60  0001 C CNN
@@
 BATT
 Wire Wire Line
-	4995 5065 4995 5180
+	4995 5060 4995 5180
 $Comp
 L SW_Push SW1
@@
 	4995 5580 4995 5660
 $Comp
-L R R9
+L R R8
 U 1 1 5B0485D5
 P 4995 5810
-F 0 "R9" V 5075 5810 50  0000 C CNN
+F 0 "R8" V 5075 5810 50  0000 C CNN
 F 1 "R" V 4995 5810 50  0000 C CNN
 F 2 "Resistors_SMD:R_1206_HandSoldering" V 4925 5810 50  0001 C CNN
@@
 Connection ~ 3765 2020
 $Comp
-L R R6
+L R R5
 U 1 1 5B04EEFE
 P 3765 2245
-F 0 "R6" V 3845 2245 50  0000 C CNN
+F 0 "R5" V 3845 2245 50  0000 C CNN
 F 1 "R" V 3765 2245 50  0000 C CNN
 F 2 "Resistors_SMD:R_1206_HandSoldering" V 3695 2245 50  0001 C CNN
@@
 Connection ~ 3570 1270
 $Comp
-L R R5
+L R R4
 U 1 1 5B04F4C7
 P 3570 945
-F 0 "R5" V 3650 945 50  0000 C CNN
+F 0 "R4" V 3650 945 50  0000 C CNN
 F 1 "R" V 3570 945 50  0000 C CNN
 F 2 "Resistors_SMD:R_1206_HandSoldering" V 3500 945 50  0001 C CNN
@@
 Wire Wire Line
 	6585 5065 6585 5340
-NoConn ~ 6685 5065
-NoConn ~ 6785 5065
-NoConn ~ 6885 5065
-NoConn ~ 6985 5065
 $Comp
 L GND #PWR016
@@
 EN1_A
 Wire Wire Line
-	1985 5710 1275 5710
+	1275 5710 1985 5710
 Text GLabel 1275 5710 0    60   Input ~ 0
 IN1_A
@@
 $EndComp
 Wire Wire Line
-	1985 6460 1310 6460
+	1310 6460 1985 6460
 Text GLabel 1310 6460 0    60   Input ~ 0
 IN2_A
@@
 Connection ~ 1445 6460
 $Comp
-L R R4
+L R R3
 U 1 1 5B0572B7
 P 1445 6675
-F 0 "R4" V 1525 6675 50  0000 C CNN
+F 0 "R3" V 1525 6675 50  0000 C CNN
 F 1 "R" V 1445 6675 50  0000 C CNN
 F 2 "Resistors_SMD:R_1206_HandSoldering" V 1375 6675 50  0001 C CNN
@@
 Connection ~ 3815 5710
 $Comp
-L R R7
+L R R6
 U 1 1 5B058343
 P 3815 5465
-F 0 "R7" V 3895 5465 50  0000 C CNN
+F 0 "R6" V 3895 5465 50  0000 C CNN
 F 1 "R" V 3815 5465 50  0000 C CNN
 F 2 "Resistors_SMD:R_1206_HandSoldering" V 3745 5465 50  0001 C CNN
@@
 Connection ~ 4080 6460
 $Comp
-L R R8
+L R R7
 U 1 1 5B058D90
 P 4080 6720
-F 0 "R8" V 4160 6720 50  0000 C CNN
+F 0 "R7" V 4160 6720 50  0000 C CNN
 F 1 "R" V 4080 6720 50  0000 C CNN
 F 2 "Resistors_SMD:R_1206_HandSoldering" V 4010 6720 50  0001 C CNN
@@
 	1    0    0    -1
 $EndComp
+$Comp
+L Conn_01x16_Female J5
+U 1 1 5B053A6F
+P 5785 4865
+F 0 "J5" H 5785 5665 50  0000 C CNN
+F 1 "Conn_01x16_Female" H 5785 3965 50  0000 C CNN
+F 2 "Socket_Strips:Socket_Strip_Straight_1x16_Pitch2.54mm" H 5785 4865 50  0001 C CNN
+F 3 "" H 5785 4865 50  0001 C CNN
+	1    5785 4865
+	0    -1   -1   0
+$EndComp
+Text GLabel 4205 3225 0    60   Input ~ 0
+3v3_gyro
+Text GLabel 4750 5060 0    60   Input ~ 0
+3v3_gyro
+Wire Wire Line
+	4750 5060 4995 5065
+Wire Wire Line
+	4995 5065 5085 5065
 $EndSCHEMATC

Commit message: updated
Parts:
- removed R11, R3, R5, R7: R, Resistors_SMD:R_1206_HandSoldering, symbol R
Connections:
- wire segments 131 -> 123
Other:
- moved on the sheet: R10, R2, R4, R6
Changed lines of the file:
@@
 Text GLabel 8755 2270 0    60   Input ~ 0
 DATA2
-Wire Wire Line
-	3765 2020 3765 2095
-Connection ~ 3765 2020
-$Comp
-L R R5
-U 1 1 5B04EEFE
-P 3765 2245
-F 0 "R5" V 3845 2245 50  0000 C CNN
-F 1 "R" V 3765 2245 50  0000 C CNN
-F 2 "Resistors_SMD:R_1206_HandSoldering" V 3695 2245 50  0001 C CNN
-F 3 "" H 3765 2245 50  0001 C CNN
-	1    3765 2245
-	1    0    0    -1
-$EndComp
-Wire Wire Line
-	3765 2395 3765 2435
-$Comp
-L GND #PWR012
-U 1 1 5B04F09F
-P 3765 2435
-F 0 "#PWR012" H 3765 2185 50  0001 C CNN
-F 1 "GND" H 3765 2285 50  0000 C CNN
-F 2 "" H 3765 2435 50  0001 C CNN
-F 3 "" H 3765 2435 50  0001 C CNN
-	1    3765 2435
-	0    -1   -1   0
-$EndComp
-Wire Wire Line
-	3570 1270 3570 1095
-Connection ~ 3570 1270
 $Comp
 L R R4
 U 1 1 5B04F4C7
-P 3570 945
-F 0 "R4" V 3650 945 50  0000 C CNN
-F 1 "R" V 3570 945 50  0000 C CNN
-F 2 "Resistors_SMD:R_1206_HandSoldering" V 3500 945 50  0001 C CNN
-F 3 "" H 3570 945 50  0001 C CNN
-	1    3570 945
-	1    0    0    -1
-$EndComp
-Wire Wire Line
-	3570 795  3570 720
-$Comp
-L GND #PWR013
+P 4080 795
+F 0 "R4" V 4160 795 50  0000 C CNN
+F 1 "R" V 4080 795 50  0000 C CNN
+F 2 "Resistors_SMD:R_1206_HandSoldering" V 4010 795 50  0001 C CNN
+F 3 "" H 4080 795 50  0001 C CNN
+	1    4080 795
+	1    0    0    -1
+$EndComp
+Wire Wire Line
+	4080 645  4080 570
+$Comp
+L GND #PWR012
 U 1 1 5B04F60A
-P 3570 720
-F 0 "#PWR013" H 3570 470 50  0001 C CNN
-F 1 "GND" H 3570 570 50  0000 C CNN
-F 2 "" H 3570 720 50  0001 C CNN
-F 3 "" H 3570 720 50  0001 C CNN
-	1    3570 720
+P 4080 570
+F 0 "#PWR012" H 4080 320 50  0001 C CNN
+F 1 "GND" H 4080 420 50  0000 C CNN
+F 2 "" H 4080 570 50  0001 C CNN
+F 3 "" H 4080 570 50  0001 C CNN
+	1    4080 570
 	0    -1   -1   0
 $EndComp
-Wire Wire Line
-	6185 2065 6185 2210
-Connection ~ 6185 2065
-$Comp
-L R R11
-U 1 1 5B04FBC0
-P 6185 2360
-F 0 "R11" V 6265 2360 50  0000 C CNN
-F 1 "R" V 6185 2360 50  0000 C CNN
-F 2 "Resistors_SMD:R_1206_HandSoldering" V 6115 2360 50  0001 C CNN
-F 3 "" H 6185 2360 50  0001 C CNN
-	1    6185 2360
-	1    0    0    -1
-$EndComp
-Wire Wire Line
-	6185 2510 6185 2555
-$Comp
-L GND #PWR014
-U 1 1 5B04FDC4
-P 6185 2555
-F 0 "#PWR014" H 6185 2305 50  0001 C CNN
-F 1 "GND" H 6185 2405 50  0000 C CNN
-F 2 "" H 6185 2555 50  0001 C CNN
-F 3 "" H 6185 2555 50  0001 C CNN
-	1    6185 2555
-	0    -1   -1   0
-$EndComp
-Wire Wire Line
-	6175 1270 6175 1160
-Connection ~ 6175 1270
 $Comp
 L R R10
 U 1 1 5B0501E5
-P 6175 1010
-F 0 "R10" V 6255 1010 50  0000 C CNN
-F 1 "R" V 6175 1010 50  0000 C CNN
-F 2 "Resistors_SMD:R_1206_HandSoldering" V 6105 1010 50  0001 C CNN
-F 3 "" H 6175 1010 50  0001 C CNN
-	1    6175 1010
-	1    0    0    -1
-$EndComp
-Wire Wire Line
-	6175 860  6175 755
-$Comp
-L GND #PWR015
+P 5710 2400
+F 0 "R10" V 5790 2400 50  0000 C CNN
+F 1 "R" V 5710 2400 50  0000 C CNN
+F 2 "Resistors_SMD:R_1206_HandSoldering" V 5640 2400 50  0001 C CNN
+F 3 "" H 5710 2400 50  0001 C CNN
+	1    5710 2400
+	-1   0    0    1
+$EndComp
+Wire Wire Line
+	5710 2550 5710 2655
+$Comp
+L GND #PWR013
 U 1 1 5B0503F8
-P 6175 755
-F 0 "#PWR015" H 6175 505 50  0001 C CNN
-F 1 "GND" H 6175 605 50  0000 C CNN
-F 2 "" H 6175 755 50  0001 C CNN
-F 3 "" H 6175 755 50  0001 C CNN
-	1    6175 755
-	0    -1   -1   0
+P 5710 2655
+F 0 "#PWR013" H 5710 2405 50  0001 C CNN
+F 1 "GND" H 5710 2505 50  0000 C CNN
+F 2 "" H 5710 2655 50  0001 C CNN
+F 3 "" H 5710 2655 50  0001 C CNN
+	1    5710 2655
+	0    1    1    0
 $EndComp
 Wire Wire Line
@@
 	6585 5065 6585 5340
 $Comp
-L GND #PWR016
+L GND #PWR014
 U 1 1 5B052D8A
 P 6585 5340
-F 0 "#PWR016" H 6585 5090 50  0001 C CNN
+F 0 "#PWR014" H 6585 5090 50  0001 C CNN
 F 1 "GND" H 6585 5190 50  0000 C CNN
 F 2 "" H 6585 5340 50  0001 C CNN
@@
 	5295 910  5245 910
 $Comp
-L GND #PWR017
+L GND #PWR015
 U 1 1 5B054309
 P 5245 910
-F 0 "#PWR017" H 5245 660 50  0001 C CNN
+F 0 "#PWR015" H 5245 660 50  0001 C CNN
 F 1 "GND" H 5245 760 50  0000 C CNN
 F 2 "" H 5245 910 50  0001 C CNN
@@
 EN1_A
 $Comp
-L GND #PWR018
+L GND #PWR016
 U 1 1 5B0559FD
 P 3610 6160
-F 0 "#PWR018" H 3610 5910 50  0001 C CNN
+F 0 "#PWR016" H 3610 5910 50  0001 C CNN
 F 1 "GND" H 3610 6010 50  0000 C CNN
 F 2 "" H 3610 6160 50  0001 C CNN
@@
 IN1_A
 Wire Wire Line
-	1370 5710 1370 5610
-Connection ~ 1370 5710
+	1965 5435 1965 5560
 $Comp
 L R R2
 U 1 1 5B056857
-P 1370 5460
-F 0 "R2" V 1450 5460 50  0000 C CNN
-F 1 "R" V 1370 5460 50  0000 C CNN
-F 2 "Resistors_SMD:R_1206_HandSoldering" V 1300 5460 50  0001 C CNN
-F 3 "" H 1370 5460 50  0001 C CNN
-	1    1370 5460
-	1    0    0    -1
-$EndComp
-Wire Wire Line
-	1370 5310 1370 5275
-$Comp
-L GND #PWR019
+P 1965 5285
+F 0 "R2" V 2045 5285 50  0000 C CNN
+F 1 "R" V 1965 5285 50  0000 C CNN
+F 2 "Resistors_SMD:R_1206_HandSoldering" V 1895 5285 50  0001 C CNN
+F 3 "" H 1965 5285 50  0001 C CNN
+	1    1965 5285
+	1    0    0    -1
+$EndComp
+Wire Wire Line
+	1965 5135 1965 5100
+$Comp
+L GND #PWR017
 U 1 1 5B056B60
-P 1370 5275
-F 0 "#PWR019" H 1370 5025 50  0001 C CNN
-F 1 "GND" H 1370 5125 50  0000 C CNN
-F 2 "" H 1370 5275 50  0001 C CNN
-F 3 "" H 1370 5275 50  0001 C CNN
-	1    1370 5275
+P 1965 5100
+F 0 "#PWR017" H 1965 4850 50  0001 C CNN
+F 1 "GND" H 1965 4950 50  0000 C CNN
+F 2 "" H 1965 5100 50  0001 C CNN
+F 3 "" H 1965 5100 50  0001 C CNN
+	1    1965 5100
 	-1   0    0    1
 $EndComp
-Wire Wire Line
-	1310 6460 1985 6460
 Text GLabel 1310 6460 0    60   Input ~ 0
 IN2_A
-Wire Wire Line
-	1445 6460 1445 6525
-Connection ~ 1445 6460
-$Comp
-L R R3
-U 1 1 5B0572B7
-P 1445 6675
-F 0 "R3" V 1525 6675 50  0000 C CNN
-F 1 "R" V 1445 6675 50  0000 C CNN
-F 2 "Resistors_SMD:R_1206_HandSoldering" V 1375 6675 50  0001 C CNN
-F 3 "" H 1445 6675 50  0001 C CNN
-	1    1445 6675
-	1    0    0    -1
-$EndComp
-Wire Wire Line
-	1445 6825 1445 6860
-$Comp
-L GND #PWR020
-U 1 1 5B05758C
-P 1445 6860
-F 0 "#PWR020" H 1445 6610 50  0001 C CNN
-F 1 "GND" H 1445 6710 50  0000 C CNN
-F 2 "" H 1445 6860 50  0001 C CNN
-F 3 "" H 1445 6860 50  0001 C CNN
-	1    1445 6860
-	1    0    0    -1
-$EndComp
 Wire Wire Line
 	3485 5710 3945 5710
 Text GLabel 3945 5710 2    60   Input ~ 0
 IN4_A
-Wire Wire Line
-	3815 5710 3815 5615
-Connection ~ 3815 5710
 $Comp
 L R R6
 U 1 1 5B058343
-P 3815 5465
-F 0 "R6" V 3895 5465 50  0000 C CNN
-F 1 "R" V 3815 5465 50  0000 C CNN
-F 2 "Resistors_SMD:R_1206_HandSoldering" V 3745 5465 50  0001 C CNN
-F 3 "" H 3815 5465 50  0001 C CNN
-	1    3815 5465
-	1    0    0    -1
-$EndComp
-Wire Wire Line
-	3815 5315 3815 5280
-$Comp
-L GND #PWR021
+P 3530 6840
+F 0 "R6" V 3610 6840 50  0000 C CNN
+F 1 "R" V 3530 6840 50  0000 C CNN
+F 2 "Resistors_SMD:R_1206_HandSoldering" V 3460 6840 50  0001 C CNN
+F 3 "" H 3530 6840 50  0001 C CNN
+	1    3530 6840
+	-1   0    0    1
+$EndComp
+Wire Wire Line
+	3530 6990 3530 7025
+$Comp
+L GND #PWR018
 U 1 1 5B05857D
-P 3815 5280
-F 0 "#PWR021" H 3815 5030 50  0001 C CNN
-F 1 "GND" H 3815 5130 50  0000 C CNN
-F 2 "" H 3815 5280 50  0001 C CNN
-F 3 "" H 3815 5280 50  0001 C CNN
-	1    3815 5280
-	-1   0    0    1
+P 3530 7025
+F 0 "#PWR018" H 3530 6775 50  0001 C CNN
+F 1 "GND" H 3530 6875 50  0000 C CNN
+F 2 "" H 3530 7025 50  0001 C CNN
+F 3 "" H 3530 7025 50  0001 C CNN
+	1    3530 7025
+	1    0    0    -1
 $EndComp
 Wire Wire Line
@@
 Text GLabel 4160 6460 2    60   Input ~ 0
 IN3_A
-Wire Wire Line
-	4080 6460 4080 6570
-Connection ~ 4080 6460
-$Comp
-L R R7
-U 1 1 5B058D90
-P 4080 6720
-F 0 "R7" V 4160 6720 50  0000 C CNN
-F 1 "R" V 4080 6720 50  0000 C CNN
-F 2 "Resistors_SMD:R_1206_HandSoldering" V 4010 6720 50  0001 C CNN
-F 3 "" H 4080 6720 50  0001 C CNN
-	1    4080 6720
-	1    0    0    -1
-$EndComp
-Wire Wire Line
-	4080 6870 4080 6905
-$Comp
-L GND #PWR022
-U 1 1 5B058F9A
-P 4080 6905
-F 0 "#PWR022" H 4080 6655 50  0001 C CNN
-F 1 "GND" H 4080 6755 50  0000 C CNN
-F 2 "" H 4080 6905 50  0001 C CNN
-F 3 "" H 4080 6905 50  0001 C CNN
-	1    4080 6905
-	1    0    0    -1
-$EndComp
 $Comp
 L Conn_01x16_Female J5
@@
 Wire Wire Line
 	4995 5065 5085 5065
+Wire Wire Line
+	4080 945  4080 1120
+Connection ~ 4080 1120
+Wire Wire Line
+	5710 2250 5710 2210
+Connection ~ 5710 2210
+Wire Wire Line
+	1310 6460 1985 6460
+Connection ~ 1965 5560
+Wire Wire Line
+	3530 6690 3530 6610
+Connection ~ 3530 6610
 $EndSCHEMATC

Commit message: final version
added silkscreen
Changed lines of the file:
@@
 Wire Wire Line
 	6995 3990 6995 3900
+Text GLabel 6485 3970 1    60   Input ~ 0
+IN2_B
 Text GLabel 5885 3965 1    60   Input ~ 0
-IN2_B
-Text GLabel 6485 3970 1    60   Input ~ 0
 EN1_B
 Text GLabel 6085 3970 1    60   Input ~ 0
